Commit message: Load model temporarily but with extra grippers

File: src/dual_ur3e_description/urdf/dual_ur3e.urdf.xacro (robot description, xacro)
@@ -1,29 +1,9 @@
 <?xml version="1.0"?>
 <robot xmlns:xacro="http://www.ros.org/wiki/xacro" name="dual_ur3e_with_grippers">
-  <!-- 导入UR宏定义（不是主文件） -->
+  <!-- 导入UR宏定义 -->
   <xacro:include filename="$(find ur_description)/urdf/ur_macro.xacro"/>
   <!-- 导入Robotiq夹爪宏定义 -->
   <xacro:include filename="$(find robotiq_85_description)/urdf/robotiq_85_gripper.urdf.xacro"/>
-  <!-- 基座平台 -->
-  <link name="base_platform">
-    <visual>
-      <geometry>
-        <box size="2.0 1.5 0.1"/>
-      </geometry>
-      <material name="gray">
-        <color rgba="0.5 0.5 0.5 1.0"/>
-      </material>
-    </visual>
-    <collision>
-      <geometry>
-        <box size="2.0 1.5 0.1"/>
-      </geometry>
-    </collision>
-    <inertial>
-      <mass value="100"/>
-      <inertia ixx="10" ixy="0" ixz="0" iyy="10" iyz="0" izz="10"/>
-    </inertial>
-  </link>
-  <!-- 左臂UR3e - 自动创建world并连接到它 -->
+  <!-- 左臂UR3e -->
   <xacro:ur_robot
     name="left_arm"
@@ -38,17 +18,11 @@
     safety_pos_margin="0.15"
     safety_k_position="20">
-    <origin xyz="-0.5 0.3 0.05" rpy="0 0 0"/>
+    <origin xyz="0 0.4 0" rpy="0 0 0"/>
   </xacro:ur_robot>
-  <!-- 将基座平台连接到world（由左臂创建） -->
-  <joint name="world_to_platform" type="fixed">
-    <parent link="world"/>
-    <child link="base_platform"/>
-    <origin xyz="0 0 0.05" rpy="0 0 0"/>
-  </joint>
-  <!-- 右臂UR3e - 连接到基座平台而不是world -->
+  <!-- 右臂UR3e -->
   <xacro:ur_robot
     name="right_arm"
     tf_prefix="right_"
-    parent="base_platform"
+    parent="world"
     joint_limits_parameters_file="$(find ur_description)/config/ur3e/joint_limits.yaml"
     kinematics_parameters_file="$(find ur_description)/config/ur3e/default_kinematics.yaml"
@@ -59,13 +33,13 @@
     safety_pos_margin="0.15"
     safety_k_position="20">
-    <origin xyz="-0.5 -0.3 0.05" rpy="0 0 0"/>
+    <origin xyz="0 -0.4 0" rpy="0 0 0"/>
   </xacro:ur_robot>
-  <!-- 左臂夹爪 -->
+  <!-- 只添加左臂和右臂的夹爪，不要添加独立的夹爪 -->
   <xacro:robotiq_85_gripper prefix="left_gripper_" parent="left_tool0">
     <origin xyz="0 0 0" rpy="0 0 0"/>
   </xacro:robotiq_85_gripper>
-  <!-- 右臂夹爪 -->
   <xacro:robotiq_85_gripper prefix="right_gripper_" parent="right_tool0">
     <origin xyz="0 0 0" rpy="0 0 0"/>
   </xacro:robotiq_85_gripper>
+  <!-- 注意：这里不要包含没有前缀的robotiq夹爪！ -->
 </robot>

Commit message: Basic model structure correct

File: src/dual_ur3e_description/urdf/dual_ur3e.urdf.xacro (robot description, xacro)
@@ -1,45 +1,134 @@
 <?xml version="1.0"?>
-<robot xmlns:xacro="http://www.ros.org/wiki/xacro" name="dual_ur3e_with_grippers">
-  <!-- 导入UR宏定义 -->
+<robot xmlns:xacro="http://ros.org/wiki/xacro" name="dual_arm_robot">
+  <!-- Import Xacro macros -->
   <xacro:include filename="$(find ur_description)/urdf/ur_macro.xacro"/>
-  <!-- 导入Robotiq夹爪宏定义 -->
-  <xacro:include filename="$(find robotiq_85_description)/urdf/robotiq_85_gripper.urdf.xacro"/>
-  <!-- 左臂UR3e -->
+  <xacro:include filename="$(find robotiq_85_description)/urdf/robotiq_85_gripper_macro.urdf.xacro"/>
+  <!-- World frame -->
+  <link name="world"/>
+  <!-- Base table - 2m x 2m  -->
+  <joint name="world_to_table" type="fixed">
+    <parent link="world"/>
+    <child link="table_link"/>
+    <origin xyz="0 0 0" rpy="0 0 0"/>
+  </joint>
+  <link name="table_link">
+    <visual>
+      <origin xyz="0 0 0.75" rpy="0 0 0"/>
+      <geometry>
+        <box size="2.0 2.0 0.05"/>
+      </geometry>
+      <material name="table_material">
+        <color rgba="0.9 0.8 0.6 1.0"/>
+      </material>
+    </visual>
+    <collision>
+      <origin xyz="0 0 0.75" rpy="0 0 0"/>
+      <geometry>
+        <box size="2.0 2.0 0.05"/>
+      </geometry>
+    </collision>
+    <inertial>
+      <mass value="30"/>
+      <origin xyz="0 0 0.75" rpy="0 0 0"/>
+      <inertia ixx="10" ixy="0" ixz="0" iyy="10" iyz="0" izz="20"/>
+    </inertial>
+  </link>
+  <!-- Left arm base mount - 位于 (0.5, 0.5) -->
+  <joint name="table_to_left_base" type="fixed">
+    <parent link="table_link"/>
+    <child link="left_base_mount"/>
+    <origin xyz="0.5 0.5 0.775" rpy="0 0 0"/>
+  </joint>
+  <link name="left_base_mount">
+    <visual>
+      <origin xyz="0 0 0.01" rpy="0 0 0"/>
+      <geometry>
+        <cylinder radius="0.08" length="0.02"/>
+      </geometry>
+      <material name="base_material">
+        <color rgba="0.3 0.3 0.3 1.0"/>
+      </material>
+    </visual>
+    <collision>
+      <origin xyz="0 0 0.01" rpy="0 0 0"/>
+      <geometry>
+        <cylinder radius="0.08" length="0.02"/>
+      </geometry>
+    </collision>
+    <inertial>
+      <mass value="2"/>
+      <origin xyz="0 0 0.01" rpy="0 0 0"/>
+      <inertia ixx="0.01" ixy="0" ixz="0" iyy="0.01" iyz="0" izz="0.01"/>
+    </inertial>
+  </link>
+  <!-- Right arm base mount - 位于 (-0.5, 0.5) -->
+  <joint name="table_to_right_base" type="fixed">
+    <parent link="table_link"/>
+    <child link="right_base_mount"/>
+    <origin xyz="-0.5 0.5 0.775" rpy="0 0 0"/>
+  </joint>
+  <link name="right_base_mount">
+    <visual>
+      <origin xyz="0 0 0.01" rpy="0 0 0"/>
+      <geometry>
+        <cylinder radius="0.08" length="0.02"/>
+      </geometry>
+      <material name="base_material">
+        <color rgba="0.3 0.3 0.3 1.0"/>
+      </material>
+    </visual>
+    <collision>
+      <origin xyz="0 0 0.01" rpy="0 0 0"/>
+      <geometry>
+        <cylinder radius="0.08" length="0.02"/>
+      </geometry>
+    </collision>
+    <inertial>
+      <mass value="2"/>
+      <origin xyz="0 0 0.01" rpy="0 0 0"/>
+      <inertia ixx="0.01" ixy="0" ixz="0" iyy="0.01" iyz="0" izz="0.01"/>
+    </inertial>
+  </link>
+  <!-- Left UR5 arm -->
   <xacro:ur_robot
-    name="left_arm"
+    name="left_ur5"
     tf_prefix="left_"
-    parent="world"
-    joint_limits_parameters_file="$(find ur_description)/config/ur3e/joint_limits.yaml"
-    kinematics_parameters_file="$(find ur_description)/config/ur3e/default_kinematics.yaml"
-    physical_parameters_file="$(find ur_description)/config/ur3e/physical_parameters.yaml"
-    visual_parameters_file="$(find ur_description)/config/ur3e/visual_parameters.yaml"
-    transmission_hw_interface=""
+    parent="left_base_mount"
+    joint_limits_parameters_file="$(find ur_description)/config/ur5/joint_limits.yaml"
+    kinematics_parameters_file="$(find ur_description)/config/ur5/default_kinematics.yaml"
+    physical_parameters_file="$(find ur_description)/config/ur5/physical_parameters.yaml"
+    visual_parameters_file="$(find ur_description)/config/ur5/visual_parameters.yaml"
     safety_limits="false"
     safety_pos_margin="0.15"
     safety_k_position="20">
-    <origin xyz="0 0.4 0" rpy="0 0 0"/>
+    <origin xyz="0 0 0.02" rpy="0 0 -1.5708"/>
   </xacro:ur_robot>
-  <!-- 右臂UR3e -->
+  <!-- Right UR5 arm -->
   <xacro:ur_robot
-    name="right_arm"
+    name="right_ur5"
     tf_prefix="right_"
-    parent="world"
-    joint_limits_parameters_file="$(find ur_description)/config/ur3e/joint_limits.yaml"
-    kinematics_parameters_file="$(find ur_description)/config/ur3e/default_kinematics.yaml"
-    physical_parameters_file="$(find ur_description)/config/ur3e/physical_parameters.yaml"
-    visual_parameters_file="$(find ur_description)/config/ur3e/visual_parameters.yaml"
-    transmission_hw_interface=""
+    parent="right_base_mount"
+    joint_limits_parameters_file="$(find ur_description)/config/ur5/joint_limits.yaml"
+    kinematics_parameters_file="$(find ur_description)/config/ur5/default_kinematics.yaml"
+    physical_parameters_file="$(find ur_description)/config/ur5/physical_parameters.yaml"
+    visual_parameters_file="$(find ur_description)/config/ur5/visual_parameters.yaml"
     safety_limits="false"
     safety_pos_margin="0.15"
     safety_k_position="20">
-    <origin xyz="0 -0.4 0" rpy="0 0 0"/>
+    <origin xyz="0 0 0.02" rpy="0 0 -1.5708"/>
   </xacro:ur_robot>
-  <!-- 只添加左臂和右臂的夹爪，不要添加独立的夹爪 -->
-  <xacro:robotiq_85_gripper prefix="left_gripper_" parent="left_tool0">
+  <!-- Left arm robotiq gripper -->
+  <xacro:robotiq_85_gripper
+    prefix="left_"
+    parent="left_tool0"
+    sim="true">
     <origin xyz="0 0 0" rpy="0 0 0"/>
   </xacro:robotiq_85_gripper>
-  <xacro:robotiq_85_gripper prefix="right_gripper_" parent="right_tool0">
+  <!-- Right arm robotiq gripper -->
+  <xacro:robotiq_85_gripper
+    prefix="right_"
+    parent="right_tool0"
+    sim="true">
     <origin xyz="0 0 0" rpy="0 0 0"/>
   </xacro:robotiq_85_gripper>
-  <!-- 注意：这里不要包含没有前缀的robotiq夹爪！ -->
 </robot>

Commit message: New model

File: src/dual_ur3e_description/urdf/dual_ur3e.urdf.xacro (robot description, xacro)
@@ -6,9 +6,9 @@
   <!-- World frame -->
   <link name="world"/>
-  <!-- Base table - 2m x 2m  -->
+  <!-- Base table - 4m x 2m  -->
   <joint name="world_to_table" type="fixed">
     <parent link="world"/>
     <child link="table_link"/>
-    <origin xyz="0 0 0" rpy="0 0 0"/>
+    <origin xyz="2.0 1.0 0" rpy="0 0 0"/>
   </joint>
   <link name="table_link">
@@ -16,5 +16,5 @@
       <origin xyz="0 0 0.75" rpy="0 0 0"/>
       <geometry>
-        <box size="2.0 2.0 0.05"/>
+        <box size="4.0 2.0 0.05"/>
       </geometry>
       <material name="table_material">
@@ -25,18 +25,18 @@
       <origin xyz="0 0 0.75" rpy="0 0 0"/>
       <geometry>
-        <box size="2.0 2.0 0.05"/>
+        <box size="4.0 2.0 0.05"/>
       </geometry>
     </collision>
     <inertial>
-      <mass value="30"/>
+      <mass value="60"/>
       <origin xyz="0 0 0.75" rpy="0 0 0"/>
-      <inertia ixx="10" ixy="0" ixz="0" iyy="10" iyz="0" izz="20"/>
+      <inertia ixx="20" ixy="0" ixz="0" iyy="40" iyz="0" izz="60"/>
     </inertial>
   </link>
-  <!-- Left arm base mount - 位于 (0.5, 0.5) -->
+  <!-- Left arm base mount - 位于 (-0.5, 0)，保持末端朝向 -X -->
   <joint name="table_to_left_base" type="fixed">
     <parent link="table_link"/>
     <child link="left_base_mount"/>
-    <origin xyz="0.5 0.5 0.775" rpy="0 0 0"/>
+    <origin xyz="-0.5 0 0.775" rpy="0 0 -1.5708"/>
   </joint>
   <link name="left_base_mount">
@@ -62,9 +62,9 @@
     </inertial>
   </link>
-  <!-- Right arm base mount - 位于 (-0.5, 0.5) -->
+  <!-- Right arm base mount - 位于 (0.5, 0)，保持末端朝向 +X -->
   <joint name="table_to_right_base" type="fixed">
     <parent link="table_link"/>
     <child link="right_base_mount"/>
-    <origin xyz="-0.5 0.5 0.775" rpy="0 0 0"/>
+    <origin xyz="0.5 0 0.775" rpy="0 0 1.5708"/>
   </joint>
   <link name="right_base_mount">
@@ -94,5 +94,5 @@
     name="left_ur5"
     tf_prefix="left_"
-    parent="left_base_mount"
+    parent="right_base_mount"
     joint_limits_parameters_file="$(find ur_description)/config/ur5/joint_limits.yaml"
     kinematics_parameters_file="$(find ur_description)/config/ur5/default_kinematics.yaml"
@@ -108,5 +108,5 @@
     name="right_ur5"
     tf_prefix="right_"
-    parent="right_base_mount"
+    parent="left_base_mount"
     joint_limits_parameters_file="$(find ur_description)/config/ur5/joint_limits.yaml"
     kinematics_parameters_file="$(find ur_description)/config/ur5/default_kinematics.yaml"

Commit message: Reduce base size

File: src/dual_ur3e_description/urdf/dual_ur3e.urdf.xacro (robot description, xacro)
@@ -6,9 +6,9 @@
   <!-- World frame -->
   <link name="world"/>
-  <!-- Base table - 4m x 2m  -->
+  <!-- Base table - 1.1m x 0.5m  -->
   <joint name="world_to_table" type="fixed">
     <parent link="world"/>
     <child link="table_link"/>
-    <origin xyz="2.0 1.0 0" rpy="0 0 0"/>
+    <origin xyz="0.55 0.25 0" rpy="0 0 0"/>
   </joint>
   <link name="table_link">
@@ -16,5 +16,5 @@
       <origin xyz="0 0 0.75" rpy="0 0 0"/>
       <geometry>
-        <box size="4.0 2.0 0.05"/>
+        <box size="1.1 0.5 0.05"/>
       </geometry>
       <material name="table_material">
@@ -25,11 +25,11 @@
       <origin xyz="0 0 0.75" rpy="0 0 0"/>
       <geometry>
-        <box size="4.0 2.0 0.05"/>
+        <box size="1.1 0.5 0.05"/>
       </geometry>
     </collision>
     <inertial>
-      <mass value="60"/>
+      <mass value="10"/>
       <origin xyz="0 0 0.75" rpy="0 0 0"/>
-      <inertia ixx="20" ixy="0" ixz="0" iyy="40" iyz="0" izz="60"/>
+      <inertia ixx="0.5" ixy="0" ixz="0" iyy="1" iyz="0" izz="1.5"/>
     </inertial>
   </link>
